File: KiCAD/Controller/Controller.kicad_sch (KiCad schematic)
At the start: 13 parts, among them U1 ST1S14PHR

Commit message: new pdfs and footprints
Parts:
- removed C1, C6: UMK325BJ106MM-T 10u, Capacitor_SMD:C_1210_3225Metric, symbol Device:C
- removed C2: 150p, symbol Device:C
- removed C3, C4, C5: 100n, Capacitor_SMD:C_0603_1608Metric, symbol Device:C
- removed C7: EKZE500ESS101MHB5D 100u, symbol Device:C_Polarized
- removed D1: STPS3L60U, symbol Device:D
- removed L1: 744314101, symbol Device:L
- removed R1: 4k7, Resistor_SMD:R_0603_1608Metric, symbol Device:R
- removed R2: 2k7, Resistor_SMD:R_0603_1608Metric, symbol Device:R
- removed R3: 47k, Resistor_SMD:R_0603_1608Metric, symbol Device:R
- removed U1: ST1S14PHR, Package_SO:TI_SO-PowerPAD-8, symbol Regulator_Switching:ST1S14PHR
- added H1, H2, H3, H4: MountingHole, MountingHole:MountingHole_3.2mm_M3, symbol Mechanical:MountingHole
Other:
- added sheet Controller (ESP32etc.kicad_sch)
- added sheet Power (power.kicad_sch)

Commit message: added some parts
Parts:
- added C13, C14: 1u, Capacitor_SMD:C_0603_1608Metric, symbol Device:C
- added J6, J7: Conn_01x03, Connector_JST:JST_XH_B3B-XH-A_1x03_P2.50mm_Vertical, symbol Connector_Generic:Conn_01x03
- added R11, R12: 100, LEDandDriver:R_0603_1608Metric_LedPrj, symbol Device:R
Connections:
- new net +12V: C13.1, C14.1, J6.1 (Pin_1), J7.1 (Pin_1)
- new net Controller/FanPWM: R11.1
- new net Controller/LEDData: R12.1
- new net FanPwmOut: J6.2 (Pin_2), R11.2
- new net GND: C13.2, C14.2, J6.3 (Pin_3), J7.3 (Pin_3)
- new net LEDDataOut: J7.2 (Pin_2), R12.2
Other:
- sheet Controller ports: added FanPWM, LEDData; removed none
