File: KiCAD/Controller/power.kicad_sch (KiCad schematic)
At the start: 14 parts, among them U1 ST1S14PHR

Commit message: added some parts
Parts:
- C1, C6: value UMK325BJ106MM-T 10u -> 10u; Manufacturer (none) -> Samsung; Manufacturer Part (none) -> CL31A106KBHNNNE
- C3, C4, C5: Manufacturer (none) -> Yageo; Manufacturer Part (none) -> CC0603KRX7R9BB104; Umax (none) -> 50V
- C7, C8: value CL31A107MQHNNNE 100uF -> 100u; Manufacturer (none) -> Samsung; Manufacturer Part (none) -> CL31A107MQHNNNE
- L1: value 744314101 -> 10u; Manufacturer (none) -> Würth; Manufacturer Part (none) -> 744314101
- R1, R2, R3: footprint Resistor_SMD:R_0603_1608Metric -> LEDandDriver:R_0603_1608Metric_LedPrj
- U1: Manufacturer (none) -> ST; Manufacturer Part (none) -> ST1S14PHR

Commit message: layout controller finished!
Parts:
- added C15, C16: 10u, Capacitor_SMD:C_1210_3225Metric, symbol Device:C
- added D4: LED, LED_SMD:LED_0603_1608Metric, symbol Device:LED
- added J8: Conn_01x03, Connector_JST:JST_XH_B3B-XH-A_1x03_P2.50mm_Vertical, symbol Connector_Generic:Conn_01x03
- added L2: 33u, Inductor_SMD:L_CommonModeChoke_Bourns_SRF1260, symbol Device:L_Coupled
- added R15: 3k, LEDandDriver:R_0603_1608Metric_LedPrj, symbol Device:R
- R1: value 4k7 -> 5k1
- R2: value 2k7 -> 3k
- R3: value 47k -> 10k
Connections:
- net +12V: now also C16.1, L2.4
- net +3.3V: now also R15.1
- net GND: now also C16.2, D4.1 (K), L2.3
- new net: D4.2 (A), R15.2
- new net Power_12V+: C15.1, J8.1 (Pin_1), L2.2
- new net Power_12V-: C15.2, J8.3 (Pin_3), L2.1
