File: KiCAD/Controller/Controller.kicad_pcb (KiCad board)
At the start: 2 copper layers, 24 parts, among them J1 Conn_01x04, J2 Conn_01x04, J3 USB_C_Receptacle_USB2.0_16P, J4 Conn_01x02, J5 Conn_01x02, U1 ST1S14PHR, U2 ESP32_C6_Wroom_1-N8

Commit message: added some parts
Parts:
- added C10: 1u, Capacitor_SMD:C_0603_1608Metric, F.Cu at (80.0, 118.9)
- added C11: 100n, Capacitor_SMD:C_0603_1608Metric, F.Cu at (80.0, 121.4)
- added C12: 100n, Capacitor_SMD:C_0603_1608Metric, F.Cu at (80.0, 123.9)
- added C13: 1u, Capacitor_SMD:C_0603_1608Metric, F.Cu at (92.0, 101.3)
- added C14: 1u, Capacitor_SMD:C_0603_1608Metric, F.Cu at (92.0, 103.8)
- added C4: 100n, Capacitor_SMD:C_0603_1608Metric, F.Cu at (95.7, 118.9)
- added C5: 100n, Capacitor_SMD:C_0603_1608Metric, F.Cu at (95.7, 121.4)
- added C9: 100u, Capacitor_SMD:C_1206_3216Metric, F.Cu at (88.8, 119.3)
- added D2: BAT54J, Diode_SMD:D_SOD-323F, F.Cu at (88.2, 122.4)
- added J6: Conn_01x03, Connector_JST:JST_XH_B3B-XH-A_1x03_P2.50mm_Vertical, F.Cu at (81.5, 103.4)
- added J7: Conn_01x03, Connector_JST:JST_XH_B3B-XH-A_1x03_P2.50mm_Vertical, F.Cu at (81.5, 111.2)
- added R10: 5k, LEDandDriver:R_0603_1608Metric_LedPrj, F.Cu at (84.0, 128.9)
- added R11: 100, LEDandDriver:R_0603_1608Metric_LedPrj, F.Cu at (92.0, 106.3)
- added R12: 100, LEDandDriver:R_0603_1608Metric_LedPrj, F.Cu at (92.0, 108.8)
- added R4: 0R, LEDandDriver:R_0603_1608Metric_LedPrj, F.Cu at (80.0, 126.4)
- added R5: 10k, LEDandDriver:R_0603_1608Metric_LedPrj, F.Cu at (80.0, 128.9)
- added R6: 10k, LEDandDriver:R_0603_1608Metric_LedPrj, F.Cu at (84.0, 118.9)
- added R7: 0R, LEDandDriver:R_0603_1608Metric_LedPrj, F.Cu at (84.0, 121.4)
- added R8: 0R, LEDandDriver:R_0603_1608Metric_LedPrj, F.Cu at (84.0, 123.9)
- added R9: 5k, LEDandDriver:R_0603_1608Metric_LedPrj, F.Cu at (84.0, 126.4)
- C1, C6: value UMK325BJ106MM-T 10u -> 10u
- C7, C8: value CL31A107MQHNNNE 100uF -> 100u
- L1: value 744314101 -> 10u
- R1, R2, R3: footprint Resistor_SMD:R_0603_1608Metric -> LEDandDriver:R_0603_1608Metric_LedPrj
Connections:
- J1 pad 1: unconnected-(J1-Pin_1-Pad1) -> +3.3V
- J1 pad 2: unconnected-(J1-Pin_2-Pad2) -> Net-(J1-Pin_2)
- J1 pad 3: unconnected-(J1-Pin_3-Pad3) -> Net-(J1-Pin_3)
- J1 pad 4: unconnected-(J1-Pin_4-Pad4) -> GND
- J2 pad 1: unconnected-(J2-Pin_1-Pad1) -> /Controller/TDO
- J2 pad 2: unconnected-(J2-Pin_2-Pad2) -> /Controller/TCK
- J2 pad 3: unconnected-(J2-Pin_3-Pad3) -> /Controller/TDI
- J2 pad 4: unconnected-(J2-Pin_4-Pad4) -> /Controller/TMS
- J3 pad A1: Net-(J3-GND-PadA1) -> GND
- J3 pad A12: Net-(J3-GND-PadA1) -> GND
- J3 pad A5: unconnected-(J3-CC1-PadA5) -> Net-(J3-CC1)
- J3 pad B1: Net-(J3-GND-PadA1) -> GND
- J3 pad B12: Net-(J3-GND-PadA1) -> GND
- J3 pad B5: unconnected-(J3-CC2-PadB5) -> Net-(J3-CC2)
- J3 pad SH: unconnected-(J3-SHIELD-PadSH) -> GND
- J4 pad 1: unconnected-(J4-Pin_1-Pad1) -> Net-(J4-Pin_1)
- J4 pad 2: unconnected-(J4-Pin_2-Pad2) -> GND
- U2 pad 10: unconnected-(U2-IO8-Pad10) -> Net-(U2-IO8)
- U2 pad 13: unconnected-(U2-IO12-Pad13) -> Net-(U2-IO12)
- U2 pad 14: unconnected-(U2-IO13-Pad14) -> Net-(U2-IO13)
- U2 pad 15: unconnected-(U2-IO9-Pad15) -> Net-(J4-Pin_1)
- U2 pad 17: unconnected-(U2-IO19-Pad17) -> /Controller/LEDData
- U2 pad 19: unconnected-(U2-IO21-Pad19) -> /Controller/FanPWM
- U2 pad 21: unconnected-(U2-IO23-Pad21) -> /Power/PowerGood
- U2 pad 24: unconnected-(U2-RXD0-Pad24) -> Net-(J1-Pin_3)
- U2 pad 25: unconnected-(U2-TXD0-Pad25) -> Net-(J1-Pin_2)
- U2 pad 3: unconnected-(U2-EN-Pad3) -> Net-(U2-EN)
- U2 pad 4: unconnected-(U2-IO4-Pad4) -> /Controller/TMS
- U2 pad 5: unconnected-(U2-IO5-Pad5) -> /Controller/TDI
- U2 pad 6: unconnected-(U2-IO6-Pad6) -> /Controller/TCK
- U2 pad 7: unconnected-(U2-IO7-Pad7) -> /Controller/TDO

Commit message: layout controller finished!
Parts:
- removed the C4 at (49.3, 78.0)
- removed the C4 at (95.7, 118.9)
- removed the C5 at (95.7, 121.4)
- removed the C5 at (49.3, 80.5)
- removed J5: Conn_01x02, Connector_PinHeader_2.54mm:PinHeader_1x02_P2.54mm_Vertical_SMD_Pin1Left
- added C15: 10u, Capacitor_SMD:C_1210_3225Metric, F.Cu at (60.8, 89.2)
- added C16: 10u, Capacitor_SMD:C_1210_3225Metric, F.Cu at (60.8, 70.2)
- added C4: 100n, Capacitor_SMD:C_0603_1608Metric, F.Cu at (86.5, 94.3)
- added C5: 100n, Capacitor_SMD:C_0603_1608Metric, F.Cu at (88.5, 94.3)
- added D3: LED, LED_SMD:LED_0603_1608Metric, F.Cu at (76.5, 65.2)
- added D4: LED, LED_SMD:LED_0603_1608Metric, F.Cu at (71.5, 80.6)
- added J8: Conn_01x03, Connector_JST:JST_XH_B3B-XH-A_1x03_P2.50mm_Vertical, F.Cu at (61.5, 96.5)
- added L2: 33u, Inductor_SMD:L_CommonModeChoke_Bourns_SRF1260, F.Cu at (60.8, 79.2)
- added R13: 0R, LEDandDriver:R_0603_1608Metric_LedPrj, F.Cu at (52.7, 53.5)
- added R14: 3k, LEDandDriver:R_0603_1608Metric_LedPrj, F.Cu at (73.3, 65.2)
- added R15: 3k, LEDandDriver:R_0603_1608Metric_LedPrj, F.Cu at (68.5, 83.2)
- added SW1: SW_Push, Button_Switch_THT:SW_PUSH_6mm_H5mm, F.Cu at (42.8, 58.2)
- J2: value Conn_01x04 -> Conn_02x05_Odd_Even; footprint Connector_PinHeader_2.54mm:PinHeader_1x04_P2.54mm_Vertical_SMD_Pin1Left -> Connector_PinHeader_2.54mm:PinHeader_2x05_P2.54mm_Vertical
- R1: value 4k7 -> 5k1
- R10, R9: value 5k -> 5k1
- R2: value 2k7 -> 3k
- R3: value 47k -> 10k
- U2: value ESP32_C6_Wroom_1-N8 -> ESP32-C6-WROOM-1; footprint LEDandDriver:ESP32-C6-WROOM-1 -> PCM_Espressif:ESP32-C6-WROOM-1
- moved J2 92.1 mm to (44.4, 66.8), turned to 90 degrees
- moved C12 85.7 mm to (50.2, 43.5), turned to 90 degrees
- moved J3 84.0 mm to (44.0, 79.8), turned to -90 degrees
- moved R8 83.9 mm to (51.1, 46.7)
- moved C9 83.4 mm to (54.7, 43.2), turned to 90 degrees
- moved C11 82.1 mm to (57.2, 42.5), turned to 90 degrees
- moved C10 80.3 mm to (52.2, 43.5), turned to 90 degrees
- moved R5 79.4 mm to (56.1, 53.2)
- moved R6 77.5 mm to (55.7, 46.7)
- moved H4 69.7 mm to (45.0, 95.0)
- moved R9 61.2 mm to (49.8, 75.6), turned to -90 degrees
- moved J1 60.0 mm to (86.3, 46.3)
- moved H1 59.3 mm to (44.5, 45.0)
- moved R10 56.6 mm to (49.8, 83.8), turned to 90 degrees
- moved R4 55.4 mm to (51.5, 78.9), turned to 180 degrees
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Connections:
- net Net-(J3-D+-PadA6) renamed /Controller/D_P
- net Net-(J3-D--PadA7) renamed /Controller/D_N
- net Net-(U2-IO12) renamed /Controller/D-
- net Net-(U2-IO13) renamed /Controller/D+
- J2 pad 1: /Controller/TDO -> +3.3V
- J2 pad 2: /Controller/TCK -> /Controller/TMS
- J2 pad 3: /Controller/TDI -> GND
- J2 pad 4: /Controller/TMS -> /Controller/TCK
- U2 pad 17: /Controller/LEDData -> /Power/PowerGood
- U2 pad 20: unconnected-(U2-IO22-Pad20) -> Net-(U2-GPIO22)
- U2 pad 21: /Power/PowerGood -> /Controller/LEDData
Routing:
- net +3.3V: track 0.00 -> 135.5 mm, vias 0 -> 4
- net +12V: track 0.00 -> 131.9 mm
- net GND: track 0.00 -> 69.9 mm, vias 0 -> 49
- net /Power/PowerGood: track 0.00 -> 45.5 mm, vias 0 -> 2
- net /Controller/LEDData: track 0.00 -> 38.6 mm
- net /Controller/TMS: track 0.00 -> 32.2 mm, vias 0 -> 2
- net Net-(U2-EN/CHIP_PU): track 0.00 -> 30.2 mm
- net /Controller/TDI: track 0.00 -> 28.8 mm, vias 0 -> 1
- net /Controller/D-: track 0.00 -> 28.6 mm
- net /Controller/D+: track 0.00 -> 28.5 mm
- net /Controller/TCK: track 0.00 -> 25.2 mm, vias 0 -> 2
- net /Controller/TDO: track 0.00 -> 19.8 mm, vias 0 -> 1
- net Net-(D2-A): track 0.00 -> 18.5 mm
- net Net-(U2-GPIO22): track 0.00 -> 15.9 mm
- net Net-(C12-Pad1): track 0.00 -> 15.2 mm
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- added copper zone on F.Cu, net +12V
- added copper zone on F.Cu, net /Power/SW
- added copper zone on B.Cu, net GND
- added copper zone on F.Cu, net GND
Other:
- board outline added: 60 x 60 mm
- board text added: "LED"
- board text added: "Lüfter"

Commit message: longer LED board
Parts:
- removed J3: USB_C_Receptacle_USB2.0_16P, Connector_USB:USB_C_Receptacle_JAE_DX07S016JA1R1500
- added USB1: HRO-TYPE-C-31-M-12, Type-C:HRO-TYPE-C-31-M-12-Assembly, F.Cu at (45.0, 79.8)
Routing:
- net GND: track 69.9 -> 78.0 mm
- net Net-(D2-A): track 18.5 -> 17.1 mm
- net /Controller/D_P: track 6.54 -> 5.71 mm
- net /Controller/D_N: track 7.18 -> 6.55 mm
