File: KiCAD/Controller/Controller.kicad_pcb (KiCad board)
At the start: 2 copper layers, 60 x 60 mm, 51 parts, among them J1 Conn_01x04, J2 Conn_02x05_Odd_Even, J4 Conn_01x02, J6 Conn_01x03, J7 Conn_01x03, J8 Conn_01x03, SW1 SW_Push, U1 ST1S14PHR, U2 ESP32-C6-WROOM-1

Commit message: added title to silkscreen
Other:
- board text added: "Bot"
- board text added: "Top"
- board text added: "enGYneer ${CURRENT_DATE} ${TITLE} v ${REVISION}"
Changed lines of the file:
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@@
 	(title_block
 		(title "Zenith Controller")
-		(date "2026-07-08")
+		(date "2026-07-23")
 		(rev "1")
 		(company "enGYneer")
@@
 		(tags "resistor")
 		(property "Reference" "R10"
-			(at -2.6 0.1 90)
+			(at 0.005 1.45 90)
 			(layer "F.SilkS")
 			(effects
@@
 		(tags "resistor")
 		(property "Reference" "R6"
-			(at -2.6 0.1 0)
+			(at 0.255 1.79 0)
 			(layer "F.SilkS")
 			(effects
@@
 		)
 		(property "Value" "10k"
-			(at 0 0.9 0)
+			(at 0.005 0.04 0)
 			(layer "F.Fab")
 			(effects
@@
 		)
 		(fp_text user "${REFERENCE}"
-			(at 0 0 0)
+			(at 0.005 1.04 0)
 			(layer "F.Fab")
 			(effects
@@
 		(tags "capacitor")
 		(property "Reference" "C11"
-			(at -3.225 0 90)
+			(at -2.765 0 90)
 			(layer "F.SilkS")
 			(effects
@@
 		)
 		(property "Value" "100n"
-			(at 3.775 0 90)
+			(at 0.235 0.005 90)
 			(layer "F.Fab")
 			(effects
@@
 		(tags "capacitor")
 		(property "Reference" "C9"
-			(at 0 -1.85 90)
+			(at -3.315 -1.245 90)
 			(layer "F.SilkS")
 			(effects
@@
 		)
 		(property "Value" "100u"
-			(at 4.5 0 90)
+			(at 0.185 0.255 90)
 			(layer "F.Fab")
 			(effects
@@
 		(tags "connector JST XH vertical")
 		(property "Reference" "J8"
-			(at 2.5 -3.55 0)
+			(at -5 0.5 0)
 			(layer "F.SilkS")
 			(effects
@@
 		(tags "capacitor")
 		(property "Reference" "C10"
-			(at 0 -1.43 90)
+			(at 2.235 -0.495 90)
 			(layer "F.SilkS")
 			(effects
@@
 		)
 		(property "Value" "1u"
-			(at 0 1.43 90)
+			(at -0.265 0.005 90)
 			(layer "F.Fab")
 			(effects
@@
 		(tags "esp32-c6")
 		(property "Reference" "U2"
-			(at 0 -17.05 0)
+			(at -1.25 13.75 0)
 			(layer "F.SilkS")
 			(effects
@@
 		(tags "capacitor")
 		(property "Reference" "C4"
-			(at 0 -1.43 90)
+			(at 2.725 0 90)
 			(layer "F.SilkS")
 			(effects
@@
 		)
 		(property "Value" "0R"
-			(at 0 0.9 0)
+			(at 0.18 0.04 0)
 			(layer "F.Fab")
 			(effects
@@
 		)
 		(fp_text user "${REFERENCE}"
-			(at 0 0 0)
+			(at -0.07 1.29 0)
 			(layer "F.Fab")
 			(effects
@@
 		(tags "capacitor")
 		(property "Reference" "C8"
-			(at 0 2 90)
+			(at -2.75 1.75 90)
 			(layer "F.SilkS")
 			(effects
@@
 		(tags "capacitor")
 		(property "Reference" "C12"
-			(at 0 -1.43 90)
+			(at 1.485 -1.495 90)
 			(layer "F.SilkS")
 			(effects
@@
 		)
 		(property "Value" "100n"
-			(at 0 1.43 90)
+			(at -0.015 0.005 90)
 			(layer "F.Fab")
 			(effects
@@
 		)
 		(property "Value" "150p"
-			(at 0 1.43 90)
+			(at 3.25 1.4 90)
 			(layer "F.Fab")
 			(effects
@@
 		(layer "Edge.Cuts")
 	)
+	(gr_text "Top"
+		(at 48.75 97.75 0)
+		(layer "F.Cu")
+		(effects
+			(font
+				(size 1 1)
+				(bold yes)
+			)
+			(justify left bottom)
+		)
+	)
+	(gr_text "Bot"
+		(at 51.5 97.75 0)
+		(layer "B.Cu")
+		(effects
+			(font
+				(size 1 1)
+				(bold yes)
+			)
+			(justify left bottom mirror)
+		)
+	)
+	(gr_text "enGYneer\n${CURRENT_DATE}\n\n${TITLE}\nv ${REVISION}"
+		(at 78.25 75 0)
+		(layer "F.SilkS")
+		(effects
+			(font
+				(size 1 1)
+				(bold yes)
+			)
+			(justify bottom)
+		)
+	)
 	(gr_text "Lüfter"
